File: CNC_New_ControlPlate/CNC_New_ControlPlate.kicad_sch (KiCad schematic)
At the start: 11 parts, among them J1 OTHER, U1 PC847

Commit message: Test
Connections:
- net 3.3V: no longer D1.38 (3V3)
- net Spindel_Dir_3.3V: no longer D1.33 (PB0)
- net Spindel_ENB_3.3V: no longer D1.34 (PB1)
- net Spindel_PWM_3.3V: no longer D1.5 (PA8)
- net X_Limit_5V: no longer D1.1 (PB12)
- net X_dir_3.3V: no longer D1.29 (PA4)
- net X_step_3.3V: no longer D1.25 (PA0)
- net Y_Limit_5V: no longer D1.2 (PB13)
- net Y_dir_3.3V: no longer D1.30 (PA5)
- net Y_step_3.3V: no longer D1.26 (PA1)
- net Z_Limit_5V: no longer D1.3 (PB14)
- net Z_dir_3.3V: no longer D1.31 (PA6)
- net Z_step_3.3V: no longer D1.27 (PA2)
Other:
- moved on the sheet: D1
Changed lines of the file:
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@@
     (stroke (width 0) (type default) (color 0 0 0 0))
   )
-  (wire (pts (xy 356.87 39.37) (xy 377.19 39.37))
+  (wire (pts (xy 355.6 40.64) (xy 377.19 39.37))
     (stroke (width 0) (type default) (color 0 0 0 0))
   )
@@
     (stroke (width 0) (type default) (color 0 0 0 0))
   )
-  (wire (pts (xy 309.88 44.45) (xy 336.55 44.45))
-    (stroke (width 0) (type default) (color 0 0 0 0))
-  )
-  (wire (pts (xy 313.69 36.83) (xy 336.55 36.83))
+  (wire (pts (xy 309.88 44.45) (xy 335.28 45.72))
+    (stroke (width 0) (type default) (color 0 0 0 0))
+  )
+  (wire (pts (xy 313.69 36.83) (xy 335.28 38.1))
     (stroke (width 0) (type default) (color 0 0 0 0))
   )
@@
     (stroke (width 0) (type default) (color 0 0 0 0))
   )
-  (wire (pts (xy 313.69 39.37) (xy 336.55 39.37))
+  (wire (pts (xy 313.69 39.37) (xy 335.28 40.64))
     (stroke (width 0) (type default) (color 0 0 0 0))
   )
@@
     (stroke (width 0) (type default) (color 0 0 0 0))
   )
-  (wire (pts (xy 317.5 67.31) (xy 336.55 67.31))
+  (wire (pts (xy 317.5 67.31) (xy 335.28 68.58))
     (stroke (width 0) (type default) (color 0 0 0 0))
   )
@@
     (stroke (width 0) (type default) (color 0 0 0 0))
   )
-  (wire (pts (xy 356.87 52.07) (xy 377.19 52.07))
+  (wire (pts (xy 355.6 53.34) (xy 377.19 52.07))
     (stroke (width 0) (type default) (color 0 0 0 0))
   )
@@
     (stroke (width 0) (type default) (color 0 0 0 0))
   )
-  (wire (pts (xy 356.87 72.39) (xy 377.19 72.39))
+  (wire (pts (xy 355.6 73.66) (xy 377.19 72.39))
     (stroke (width 0) (type default) (color 0 0 0 0))
   )
@@
     (stroke (width 0) (type default) (color 0 0 0 0))
   )
-  (wire (pts (xy 320.04 69.85) (xy 336.55 69.85))
-    (stroke (width 0) (type default) (color 0 0 0 0))
-  )
-  (wire (pts (xy 356.87 69.85) (xy 377.19 69.85))
-    (stroke (width 0) (type default) (color 0 0 0 0))
-  )
-  (wire (pts (xy 356.87 57.15) (xy 377.19 57.15))
+  (wire (pts (xy 320.04 69.85) (xy 335.28 71.12))
+    (stroke (width 0) (type default) (color 0 0 0 0))
+  )
+  (wire (pts (xy 355.6 71.12) (xy 377.19 69.85))
+    (stroke (width 0) (type default) (color 0 0 0 0))
+  )
+  (wire (pts (xy 355.6 58.42) (xy 377.19 57.15))
     (stroke (width 0) (type default) (color 0 0 0 0))
   )
@@
     (stroke (width 0) (type default) (color 0 0 0 0))
   )
-  (wire (pts (xy 356.87 59.69) (xy 377.19 59.69))
+  (wire (pts (xy 355.6 60.96) (xy 377.19 59.69))
     (stroke (width 0) (type default) (color 0 0 0 0))
   )
@@
     (stroke (width 0) (type default) (color 0 0 0 0))
   )
-  (wire (pts (xy 336.55 57.15) (xy 314.96 57.15))
+  (wire (pts (xy 335.28 58.42) (xy 314.96 57.15))
     (stroke (width 0) (type default) (color 0 0 0 0))
   )
@@
     (stroke (width 0) (type default) (color 0 0 0 0))
   )
-  (wire (pts (xy 356.87 49.53) (xy 377.19 49.53))
+  (wire (pts (xy 355.6 50.8) (xy 377.19 49.53))
     (stroke (width 0) (type default) (color 0 0 0 0))
   )
@@
     (stroke (width 0) (type default) (color 0 0 0 0))
   )
-  (wire (pts (xy 356.87 67.31) (xy 377.19 67.31))
+  (wire (pts (xy 355.6 68.58) (xy 377.19 67.31))
     (stroke (width 0) (type default) (color 0 0 0 0))
   )
@@
     (stroke (width 0) (type default) (color 0 0 0 0))
   )
-  (wire (pts (xy 313.69 34.29) (xy 336.55 34.29))
+  (wire (pts (xy 313.69 34.29) (xy 335.28 35.56))
     (stroke (width 0) (type default) (color 0 0 0 0))
   )
@@
     (stroke (width 0) (type default) (color 0 0 0 0))
   )
-  (wire (pts (xy 334.01 80.01) (xy 336.55 80.01))
-    (stroke (width 0) (type default) (color 0 0 0 0))
-  )
-  (wire (pts (xy 336.55 74.93) (xy 322.58 74.93))
+  (wire (pts (xy 334.01 80.01) (xy 335.28 81.28))
+    (stroke (width 0) (type default) (color 0 0 0 0))
+  )
+  (wire (pts (xy 335.28 76.2) (xy 322.58 74.93))
     (stroke (width 0) (type default) (color 0 0 0 0))
   )
@@
     (stroke (width 0) (type default) (color 0 0 0 0))
   )
-  (wire (pts (xy 326.39 77.47) (xy 336.55 77.47))
-    (stroke (width 0) (type default) (color 0 0 0 0))
-  )
-  (wire (pts (xy 356.87 36.83) (xy 358.14 36.83))
+  (wire (pts (xy 326.39 77.47) (xy 335.28 78.74))
+    (stroke (width 0) (type default) (color 0 0 0 0))
+  )
+  (wire (pts (xy 355.6 38.1) (xy 358.14 36.83))
     (stroke (width 0) (type default) (color 0 0 0 0))
   )
@@
     (stroke (width 0) (type default) (color 0 0 0 0))
   )
-  (wire (pts (xy 356.87 34.29) (xy 358.14 34.29))
+  (wire (pts (xy 355.6 35.56) (xy 358.14 34.29))
     (stroke (width 0) (type default) (color 0 0 0 0))
   )
@@
     (stroke (width 0) (type default) (color 0 0 0 0))
   )
-  (wire (pts (xy 356.87 62.23) (xy 377.19 62.23))
+  (wire (pts (xy 355.6 63.5) (xy 377.19 62.23))
     (stroke (width 0) (type default) (color 0 0 0 0))
   )
@@
       (effects (font (size 1.27 1.27)) hide)
     )
-    (property "Value" "" (id 1) (at 396.24 96.52 0))
+    (property "Value" "VCC" (id 1) (at 396.24 96.52 0))
     (property "Footprint" "" (id 2) (at 396.24 101.6 0)
       (effects (font (size 1.27 1.27)) hide)
@@
     (pin "9")
   )
-  (symbol (lib_id "G-LIB:BP") (at 346.71 45.72 0) (unit 1)
+  (symbol (lib_id "G-LIB:BP") (at 345.44 46.99 0) (unit 1)
     (in_bom yes) (on_board yes) (fields_autoplaced)
-    (property "Reference" "D1" (id 0) (at 346.71 27.94 0))
-    (property "Value" "BluePill" (id 1) (at 346.71 30.48 0))
-    (property "Footprint" "Module:Maple_Mini" (id 2) (at 346.71 45.72 0)
-      (effects (font (size 1.27 1.27)) hide)
-    )
-    (property "Datasheet" "" (id 3) (at 346.71 45.72 0)
+    (property "Reference" "D1" (id 0) (at 345.44 29.21 0))
+    (property "Value" "BluePill" (id 1) (at 345.44 31.75 0))
+    (property "Footprint" "Module:Maple_Mini" (id 2) (at 345.44 46.99 0)
+      (effects (font (size 1.27 1.27)) hide)
+    )
+    (property "Datasheet" "" (id 3) (at 345.44 46.99 0)
       (effects (font (size 1.27 1.27)) hide)
     )
@@
       (effects (font (size 1.27 1.27)) hide)
     )
-    (property "Value" "" (id 1) (at 396.24 92.71 0))
+    (property "Value" "GNDREF" (id 1) (at 396.24 92.71 0))
     (property "Footprint" "" (id 2) (at 396.24 87.63 0)
       (effects (font (size 1.27 1.27)) hide)

Commit message: Cancel Test
Connections:
- net 3.3V: now also D1.38 (3V3)
- net Spindel_Dir_3.3V: now also D1.33 (PB0)
- net Spindel_ENB_3.3V: now also D1.34 (PB1)
- net Spindel_PWM_3.3V: now also D1.5 (PA8)
- net X_Limit_5V: now also D1.1 (PB12)
- net X_dir_3.3V: now also D1.29 (PA4)
- net X_step_3.3V: now also D1.25 (PA0)
- net Y_Limit_5V: now also D1.2 (PB13)
- net Y_dir_3.3V: now also D1.30 (PA5)
- net Y_step_3.3V: now also D1.26 (PA1)
- net Z_Limit_5V: now also D1.3 (PB14)
- net Z_dir_3.3V: now also D1.31 (PA6)
- net Z_step_3.3V: now also D1.27 (PA2)
Other:
- moved on the sheet: D1
Changed lines of the file:
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@@
     (stroke (width 0) (type default) (color 0 0 0 0))
   )
-  (wire (pts (xy 355.6 40.64) (xy 377.19 39.37))
+  (wire (pts (xy 356.87 39.37) (xy 377.19 39.37))
     (stroke (width 0) (type default) (color 0 0 0 0))
   )
@@
     (stroke (width 0) (type default) (color 0 0 0 0))
   )
-  (wire (pts (xy 309.88 44.45) (xy 335.28 45.72))
-    (stroke (width 0) (type default) (color 0 0 0 0))
-  )
-  (wire (pts (xy 313.69 36.83) (xy 335.28 38.1))
+  (wire (pts (xy 309.88 44.45) (xy 336.55 44.45))
+    (stroke (width 0) (type default) (color 0 0 0 0))
+  )
+  (wire (pts (xy 313.69 36.83) (xy 336.55 36.83))
     (stroke (width 0) (type default) (color 0 0 0 0))
   )
@@
     (stroke (width 0) (type default) (color 0 0 0 0))
   )
-  (wire (pts (xy 313.69 39.37) (xy 335.28 40.64))
+  (wire (pts (xy 313.69 39.37) (xy 336.55 39.37))
     (stroke (width 0) (type default) (color 0 0 0 0))
   )
@@
     (stroke (width 0) (type default) (color 0 0 0 0))
   )
-  (wire (pts (xy 317.5 67.31) (xy 335.28 68.58))
+  (wire (pts (xy 317.5 67.31) (xy 336.55 67.31))
     (stroke (width 0) (type default) (color 0 0 0 0))
   )
@@
     (stroke (width 0) (type default) (color 0 0 0 0))
   )
-  (wire (pts (xy 355.6 53.34) (xy 377.19 52.07))
+  (wire (pts (xy 356.87 52.07) (xy 377.19 52.07))
     (stroke (width 0) (type default) (color 0 0 0 0))
   )
@@
     (stroke (width 0) (type default) (color 0 0 0 0))
   )
-  (wire (pts (xy 355.6 73.66) (xy 377.19 72.39))
+  (wire (pts (xy 356.87 72.39) (xy 377.19 72.39))
     (stroke (width 0) (type default) (color 0 0 0 0))
   )
@@
     (stroke (width 0) (type default) (color 0 0 0 0))
   )
-  (wire (pts (xy 320.04 69.85) (xy 335.28 71.12))
-    (stroke (width 0) (type default) (color 0 0 0 0))
-  )
-  (wire (pts (xy 355.6 71.12) (xy 377.19 69.85))
-    (stroke (width 0) (type default) (color 0 0 0 0))
-  )
-  (wire (pts (xy 355.6 58.42) (xy 377.19 57.15))
+  (wire (pts (xy 320.04 69.85) (xy 336.55 69.85))
+    (stroke (width 0) (type default) (color 0 0 0 0))
+  )
+  (wire (pts (xy 356.87 69.85) (xy 377.19 69.85))
+    (stroke (width 0) (type default) (color 0 0 0 0))
+  )
+  (wire (pts (xy 356.87 57.15) (xy 377.19 57.15))
     (stroke (width 0) (type default) (color 0 0 0 0))
   )
@@
     (stroke (width 0) (type default) (color 0 0 0 0))
   )
-  (wire (pts (xy 355.6 60.96) (xy 377.19 59.69))
+  (wire (pts (xy 356.87 59.69) (xy 377.19 59.69))
     (stroke (width 0) (type default) (color 0 0 0 0))
   )
@@
     (stroke (width 0) (type default) (color 0 0 0 0))
   )
-  (wire (pts (xy 335.28 58.42) (xy 314.96 57.15))
+  (wire (pts (xy 336.55 57.15) (xy 314.96 57.15))
     (stroke (width 0) (type default) (color 0 0 0 0))
   )
@@
     (stroke (width 0) (type default) (color 0 0 0 0))
   )
-  (wire (pts (xy 355.6 50.8) (xy 377.19 49.53))
+  (wire (pts (xy 356.87 49.53) (xy 377.19 49.53))
     (stroke (width 0) (type default) (color 0 0 0 0))
   )
@@
     (stroke (width 0) (type default) (color 0 0 0 0))
   )
-  (wire (pts (xy 355.6 68.58) (xy 377.19 67.31))
+  (wire (pts (xy 356.87 67.31) (xy 377.19 67.31))
     (stroke (width 0) (type default) (color 0 0 0 0))
   )
@@
     (stroke (width 0) (type default) (color 0 0 0 0))
   )
-  (wire (pts (xy 313.69 34.29) (xy 335.28 35.56))
+  (wire (pts (xy 313.69 34.29) (xy 336.55 34.29))
     (stroke (width 0) (type default) (color 0 0 0 0))
   )
@@
     (stroke (width 0) (type default) (color 0 0 0 0))
   )
-  (wire (pts (xy 334.01 80.01) (xy 335.28 81.28))
-    (stroke (width 0) (type default) (color 0 0 0 0))
-  )
-  (wire (pts (xy 335.28 76.2) (xy 322.58 74.93))
+  (wire (pts (xy 334.01 80.01) (xy 336.55 80.01))
+    (stroke (width 0) (type default) (color 0 0 0 0))
+  )
+  (wire (pts (xy 336.55 74.93) (xy 322.58 74.93))
     (stroke (width 0) (type default) (color 0 0 0 0))
   )
@@
     (stroke (width 0) (type default) (color 0 0 0 0))
   )
-  (wire (pts (xy 326.39 77.47) (xy 335.28 78.74))
-    (stroke (width 0) (type default) (color 0 0 0 0))
-  )
-  (wire (pts (xy 355.6 38.1) (xy 358.14 36.83))
+  (wire (pts (xy 326.39 77.47) (xy 336.55 77.47))
+    (stroke (width 0) (type default) (color 0 0 0 0))
+  )
+  (wire (pts (xy 356.87 36.83) (xy 358.14 36.83))
     (stroke (width 0) (type default) (color 0 0 0 0))
   )
@@
     (stroke (width 0) (type default) (color 0 0 0 0))
   )
-  (wire (pts (xy 355.6 35.56) (xy 358.14 34.29))
+  (wire (pts (xy 356.87 34.29) (xy 358.14 34.29))
     (stroke (width 0) (type default) (color 0 0 0 0))
   )
@@
     (stroke (width 0) (type default) (color 0 0 0 0))
   )
-  (wire (pts (xy 355.6 63.5) (xy 377.19 62.23))
+  (wire (pts (xy 356.87 62.23) (xy 377.19 62.23))
     (stroke (width 0) (type default) (color 0 0 0 0))
   )
@@
     (pin "9")
   )
-  (symbol (lib_id "G-LIB:BP") (at 345.44 46.99 0) (unit 1)
+  (symbol (lib_id "G-LIB:BP") (at 346.71 45.72 0) (unit 1)
     (in_bom yes) (on_board yes) (fields_autoplaced)
-    (property "Reference" "D1" (id 0) (at 345.44 29.21 0))
-    (property "Value" "BluePill" (id 1) (at 345.44 31.75 0))
-    (property "Footprint" "Module:Maple_Mini" (id 2) (at 345.44 46.99 0)
-      (effects (font (size 1.27 1.27)) hide)
-    )
-    (property "Datasheet" "" (id 3) (at 345.44 46.99 0)
-      (effects (font (size 1.27 1.27)) hide)
-    )
+    (property "Reference" "D1" (id 0) (at 346.71 27.94 0))
+    (property "Value" "BluePill" (id 1) (at 346.71 30.48 0))
+    (property "Footprint" "Module:Maple_Mini" (id 2) (at 346.71 45.72 0)
+      (effects (font (size 1.27 1.27)) hide)
+    )
+    (property "Datasheet" "" (id 3) (at 346.71 45.72 0)
+      (effects (font (size 1.27 1.27)) hide)
+    )
