File: CNC_New_ControlPlate/spindel.kicad_sch (KiCad schematic)
At the start: 4 parts

Commit message: [*] номиналы блокировочных конденсаторов [+] мкроконтроллер управления оборотами шпинделя [+] кнопка паузы
Parts:
- added C? (x2): 100n, Capacitor_SMD:C_0603_1608Metric_Pad1.08x0.95mm_HandSolder, symbol Device:C
- added C? (x2): 22 pF, Capacitor_SMD:C_0603_1608Metric_Pad1.08x0.95mm_HandSolder, symbol Device:C
- added R?: 10k, symbol Device:R
- added Y?: 4MHz, symbol Device:Crystal
- U?: value (none) -> ATtiny2313V-10P; footprint (none) -> Package_DIP:DIP-20_W7.62mm
Connections:
- net +5V: now also U?.20 (VCC), C?.2, R?.1
- net GNDREF: now also U?.10 (GND), C?.1, C?.1, C?.1, C?.1
- net SP_1: now also U?.19 (PB7)
- net SP_2: now also U?.18 (PB6)
- net SP_3: now also U?.17 (PB5)
- net SP_4: now also U?.16 (PB4)
- net SP_5: now also U?.15 (PB3)
- net SP_6: now also U?.14 (PB2)
- net SP_7: now also U?.13 (PB1)
- net SP_8: now also U?.12 (PB0)
- net at U?.8: now also U?.6 (PD2), U?.7 (PD3)
- net at U?.1 (PA2/~{RESET}): now also C?.2, R?.2
- net at U?.4 (PA1/XTAL2): now also C?.2, Y?.2
- net at U?.5 (PA0/XTAL1): now also C?.2, Y?.1
- no-connect marks 0 -> 7
Other:
- moved on the sheet: U?D, U?E, U?F
