File: CNC_New_ControlPlate/spindel.kicad_sch (KiCad schematic)
At the start: 10 parts

Commit message: [*] Исправлены ошибки с выходами питания. [+] Добавлены обозначения элементов
Parts:
- gave numbers to parts that had none: 8
Changed lines of the file:
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@@
   (symbol (lib_id "power:+5V") (at 138.43 39.37 0) (unit 1)
     (in_bom yes) (on_board yes) (fields_autoplaced)
-    (property "Reference" "#PWR?" (id 0) (at 138.43 43.18 0)
+    (property "Reference" "#PWR043" (id 0) (at 138.43 43.18 0)
       (effects (font (size 1.27 1.27)) hide)
     )
@@
   (symbol (lib_id "Device:C") (at 86.36 76.2 180) (unit 1)
     (in_bom yes) (on_board yes) (fields_autoplaced)
-    (property "Reference" "C?" (id 0) (at 90.17 74.9299 0)
+    (property "Reference" "C3" (id 0) (at 90.17 74.9299 0)
       (effects (font (size 1.27 1.27)) (justify right))
     )
@@
   (symbol (lib_id "Device:C") (at 129.54 41.91 90) (unit 1)
     (in_bom yes) (on_board yes) (fields_autoplaced)
-    (property "Reference" "C?" (id 0) (at 129.54 34.29 90))
+    (property "Reference" "C6" (id 0) (at 129.54 34.29 90))
     (property "Value" "100n" (id 1) (at 129.54 36.83 90))
     (property "Footprint" "Capacitor_SMD:C_0603_1608Metric_Pad1.08x0.95mm_HandSolder" (id 2) (at 133.35 40.9448 0)
@@
   (symbol (lib_id "74xx_IEEE:7406") (at 190.5 135.89 0) (mirror y) (unit 6)
     (in_bom yes) (on_board yes)
-    (property "Reference" "U?" (id 0) (at 194.31 128.27 0))
+    (property "Reference" "U3" (id 0) (at 194.31 128.27 0))
     (property "Value" "7406" (id 1) (at 190.5 130.81 0))
     (property "Footprint" "" (id 2) (at 190.5 135.89 0)
@@
   (symbol (lib_id "power:GNDREF") (at 86.36 80.01 0) (unit 1)
     (in_bom yes) (on_board yes) (fields_autoplaced)
-    (property "Reference" "#PWR?" (id 0) (at 86.36 86.36 0)
+    (property "Reference" "#PWR039" (id 0) (at 86.36 86.36 0)
       (effects (font (size 1.27 1.27)) hide)
     )
@@
   (symbol (lib_id "74xx_IEEE:7406") (at 190.5 85.09 0) (mirror y) (unit 4)
     (in_bom yes) (on_board yes)
-    (property "Reference" "U?" (id 0) (at 194.31 77.47 0))
+    (property "Reference" "U3" (id 0) (at 194.31 77.47 0))
     (property "Value" "7406" (id 1) (at 190.5 80.01 0))
     (property "Footprint" "" (id 2) (at 190.5 85.09 0)
@@
   (symbol (lib_id "power:GNDREF") (at 119.38 44.45 0) (unit 1)
     (in_bom yes) (on_board yes) (fields_autoplaced)
-    (property "Reference" "#PWR?" (id 0) (at 119.38 50.8 0)
+    (property "Reference" "#PWR042" (id 0) (at 119.38 50.8 0)
       (effects (font (size 1.27 1.27)) hide)
     )
@@
   (symbol (lib_id "power:GNDREF") (at 111.76 80.01 0) (unit 1)
     (in_bom yes) (on_board yes) (fields_autoplaced)
-    (property "Reference" "#PWR?" (id 0) (at 111.76 86.36 0)
+    (property "Reference" "#PWR041" (id 0) (at 111.76 86.36 0)
       (effects (font (size 1.27 1.27)) hide)
     )
@@
   (symbol (lib_id "power:GNDREF") (at 190.5 91.44 0) (unit 1)
     (in_bom yes) (on_board yes) (fields_autoplaced)
-    (property "Reference" "#PWR?" (id 0) (at 190.5 97.79 0)
+    (property "Reference" "#PWR046" (id 0) (at 190.5 97.79 0)
       (effects (font (size 1.27 1.27)) hide)
     )
@@
   (symbol (lib_id "power:+5V") (at 190.5 104.14 0) (unit 1)
     (in_bom yes) (on_board yes)
-    (property "Reference" "#PWR?" (id 0) (at 190.5 107.95 0)
+    (property "Reference" "#PWR047" (id 0) (at 190.5 107.95 0)
       (effects (font (size 1.27 1.27)) hide)
     )
@@
   (symbol (lib_id "power:GNDREF") (at 138.43 105.41 0) (unit 1)
     (in_bom yes) (on_board yes) (fields_autoplaced)
-    (property "Reference" "#PWR?" (id 0) (at 138.43 111.76 0)
+    (property "Reference" "#PWR044" (id 0) (at 138.43 111.76 0)
       (effects (font (size 1.27 1.27)) hide)
     )
@@
   (symbol (lib_id "Device:R") (at 86.36 46.99 0) (unit 1)
     (in_bom yes) (on_board yes) (fields_autoplaced)
-    (property "Reference" "R?" (id 0) (at 88.9 45.7199 0)
+    (property "Reference" "R11" (id 0) (at 88.9 45.7199 0)
       (effects (font (size 1.27 1.27)) (justify left))
     )
@@
   (symbol (lib_id "power:+5V") (at 86.36 40.64 0) (unit 1)
     (in_bom yes) (on_board yes) (fields_autoplaced)
-    (property "Reference" "#PWR?" (id 0) (at 86.36 44.45 0)
+    (property "Reference" "#PWR038" (id 0) (at 86.36 44.45 0)
       (effects (font (size 1.27 1.27)) hide)
     )
@@
   (symbol (lib_id "MCU_Microchip_ATtiny:ATtiny2313V-10P") (at 138.43 74.93 0) (unit 1)
     (in_bom yes) (on_board yes) (fields_autoplaced)
-    (property "Reference" "U?" (id 0) (at 140.4494 44.45 0)
+    (property "Reference" "U4" (id 0) (at 140.4494 44.45 0)
       (effects (font (size 1.27 1.27)) (justify left))
     )
@@
   (symbol (lib_id "power:+5V") (at 190.5 78.74 0) (unit 1)
     (in_bom yes) (on_board yes)
-    (property "Reference" "#PWR?" (id 0) (at 190.5 82.55 0)
+    (property "Reference" "#PWR045" (id 0) (at 190.5 82.55 0)
       (effects (font (size 1.27 1.27)) hide)
     )
@@
   (symbol (lib_id "Device:Crystal") (at 105.41 69.85 0) (unit 1)
     (in_bom yes) (on_board yes) (fields_autoplaced)
-    (property "Reference" "Y?" (id 0) (at 105.41 62.23 0))
+    (property "Reference" "Y1" (id 0) (at 105.41 62.23 0))
     (property "Value" "4MHz" (id 1) (at 105.41 64.77 0))
     (property "Footprint" "" (id 2) (at 105.41 69.85 0)
@@
   (symbol (lib_id "power:GNDREF") (at 190.5 142.24 0) (unit 1)
     (in_bom yes) (on_board yes) (fields_autoplaced)
-    (property "Reference" "#PWR?" (id 0) (at 190.5 148.59 0)
+    (property "Reference" "#PWR050" (id 0) (at 190.5 148.59 0)
       (effects (font (size 1.27 1.27)) hide)
     )
@@
   (symbol (lib_id "power:+5V") (at 190.5 129.54 0) (unit 1)
     (in_bom yes) (on_board yes)
-    (property "Reference" "#PWR?" (id 0) (at 190.5 133.35 0)
+    (property "Reference" "#PWR049" (id 0) (at 190.5 133.35 0)
       (effects (font (size 1.27 1.27)) hide)
     )
@@
   (symbol (lib_id "power:GNDREF") (at 99.06 80.01 0) (unit 1)
     (in_bom yes) (on_board yes) (fields_autoplaced)
-    (property "Reference" "#PWR?" (id 0) (at 99.06 86.36 0)
+    (property "Reference" "#PWR040" (id 0) (at 99.06 86.36 0)
       (effects (font (size 1.27 1.27)) hide)
     )
@@
   (symbol (lib_id "Device:C") (at 111.76 76.2 180) (unit 1)
     (in_bom yes) (on_board yes) (fields_autoplaced)
-    (property "Reference" "C?" (id 0) (at 115.57 74.9299 0)
+    (property "Reference" "C5" (id 0) (at 115.57 74.9299 0)
       (effects (font (size 1.27 1.27)) (justify right))
     )
@@
   (symbol (lib_id "Device:C") (at 99.06 76.2 180) (unit 1)
     (in_bom yes) (on_board yes) (fields_autoplaced)
-    (property "Reference" "C?" (id 0) (at 102.87 74.9299 0)
+    (property "Reference" "C4" (id 0) (at 102.87 74.9299 0)
       (effects (font (size 1.27 1.27)) (justify right))
     )
@@
   (symbol (lib_id "power:GNDREF") (at 190.5 116.84 0) (unit 1)
     (in_bom yes) (on_board yes) (fields_autoplaced)
-    (property "Reference" "#PWR?" (id 0) (at 190.5 123.19 0)
+    (property "Reference" "#PWR048" (id 0) (at 190.5 123.19 0)
       (effects (font (size 1.27 1.27)) hide)
     )
@@
   (symbol (lib_id "74xx_IEEE:7406") (at 190.5 110.49 0) (mirror y) (unit 5)
     (in_bom yes) (on_board yes)
-    (property "Reference" "U?" (id 0) (at 194.31 102.87 0))
+    (property "Reference" "U3" (id 0) (at 194.31 102.87 0))
     (property "Value" "7406" (id 1) (at 190.5 105.41 0))
     (property "Footprint" "" (id 2) (at 190.5 110.49 0)

Commit message: [*] Порядок выводов на разъёме Others [*] Порядок выводов на разъёме Pause [*] Порядок подключения каналов на драйвере диф. линий [+] Начата расстановка pcb схемы
Parts:
- R11: footprint (none) -> Resistor_SMD:R_0603_1608Metric
- U3: footprint (none) -> Package_DIP:DIP-14_W7.62mm_Socket
- Y1: footprint (none) -> Crystal:Crystal_HC49-4H_Vertical
Changed lines of the file:
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@@
     (property "Reference" "U3" (id 0) (at 194.31 128.27 0))
     (property "Value" "7406" (id 1) (at 190.5 130.81 0))
-    (property "Footprint" "" (id 2) (at 190.5 135.89 0)
+    (property "Footprint" "Package_DIP:DIP-14_W7.62mm_Socket" (id 2) (at 190.5 135.89 0)
       (effects (font (size 1.27 1.27)) hide)
     )
@@
     (property "Reference" "U3" (id 0) (at 194.31 77.47 0))
     (property "Value" "7406" (id 1) (at 190.5 80.01 0))
-    (property "Footprint" "" (id 2) (at 190.5 85.09 0)
+    (property "Footprint" "Package_DIP:DIP-14_W7.62mm_Socket" (id 2) (at 190.5 85.09 0)
       (effects (font (size 1.27 1.27)) hide)
     )
@@
       (effects (font (size 1.27 1.27)) (justify left))
     )
-    (property "Footprint" "" (id 2) (at 84.582 46.99 90)
+    (property "Footprint" "Resistor_SMD:R_0603_1608Metric" (id 2) (at 84.582 46.99 90)
       (effects (font (size 1.27 1.27)) hide)
     )
@@
     (property "Reference" "Y1" (id 0) (at 105.41 62.23 0))
     (property "Value" "4MHz" (id 1) (at 105.41 64.77 0))
-    (property "Footprint" "" (id 2) (at 105.41 69.85 0)
+    (property "Footprint" "Crystal:Crystal_HC49-4H_Vertical" (id 2) (at 105.41 69.85 0)
       (effects (font (size 1.27 1.27)) hide)
     )
@@
     (property "Reference" "U3" (id 0) (at 194.31 102.87 0))
     (property "Value" "7406" (id 1) (at 190.5 105.41 0))
-    (property "Footprint" "" (id 2) (at 190.5 110.49 0)
-      (effects (font (size 1.27 1.27)) hide)
-    )
+    (property "Footprint" "Package_DIP:DIP-14_W7.62mm_Socket" (id 2) (at 190.5 110.49 0)
+      (effects (font (size 1.27 1.27)) hide)
+    )

Commit message: Edit footprints
Parts:
- U3: value 7406 -> (none); footprint Package_DIP:DIP-14_W7.62mm_Socket -> (none)
- U4: value ATtiny2313V-10P -> (none); footprint Package_DIP:DIP-20_W7.62mm -> (none)
- Y1: value 4MHz -> (none); footprint Crystal:Crystal_HC49-4H_Vertical -> (none)
Changed lines of the file:
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@@
     (in_bom yes) (on_board yes)
     (property "Reference" "U3" (id 0) (at 194.31 128.27 0))
-    (property "Value" "7406" (id 1) (at 190.5 130.81 0))
-    (property "Footprint" "Package_DIP:DIP-14_W7.62mm_Socket" (id 2) (at 190.5 135.89 0)
+    (property "Value" "" (id 1) (at 190.5 130.81 0))
+    (property "Footprint" "" (id 2) (at 190.5 135.89 0)
       (effects (font (size 1.27 1.27)) hide)
     )
@@
     (in_bom yes) (on_board yes)
     (property "Reference" "U3" (id 0) (at 194.31 77.47 0))
-    (property "Value" "7406" (id 1) (at 190.5 80.01 0))
-    (property "Footprint" "Package_DIP:DIP-14_W7.62mm_Socket" (id 2) (at 190.5 85.09 0)
+    (property "Value" "" (id 1) (at 190.5 80.01 0))
+    (property "Footprint" "" (id 2) (at 190.5 85.09 0)
       (effects (font (size 1.27 1.27)) hide)
     )
@@
       (effects (font (size 1.27 1.27)) (justify left))
     )
-    (property "Value" "ATtiny2313V-10P" (id 1) (at 140.4494 46.99 0)
+    (property "Value" "" (id 1) (at 140.4494 46.99 0)
       (effects (font (size 1.27 1.27)) (justify left))
     )
-    (property "Footprint" "Package_DIP:DIP-20_W7.62mm" (id 2) (at 138.43 74.93 0)
+    (property "Footprint" "" (id 2) (at 138.43 74.93 0)
       (effects (font (size 1.27 1.27) italic) hide)
     )
@@
     (in_bom yes) (on_board yes) (fields_autoplaced)
     (property "Reference" "Y1" (id 0) (at 105.41 62.23 0))
-    (property "Value" "4MHz" (id 1) (at 105.41 64.77 0))
-    (property "Footprint" "Crystal:Crystal_HC49-4H_Vertical" (id 2) (at 105.41 69.85 0)
+    (property "Value" "" (id 1) (at 105.41 64.77 0))
+    (property "Footprint" "" (id 2) (at 105.41 69.85 0)
       (effects (font (size 1.27 1.27)) hide)
     )
@@
     (in_bom yes) (on_board yes)
     (property "Reference" "U3" (id 0) (at 194.31 102.87 0))
-    (property "Value" "7406" (id 1) (at 190.5 105.41 0))
-    (property "Footprint" "Package_DIP:DIP-14_W7.62mm_Socket" (id 2) (at 190.5 110.49 0)
-      (effects (font (size 1.27 1.27)) hide)
-    )
+    (property "Value" "" (id 1) (at 190.5 105.41 0))
+    (property "Footprint" "" (id 2) (at 190.5 110.49 0)
+      (effects (font (size 1.27 1.27)) hide)
+    )

Commit message: [*] Разводка платы в один слой (осталось 7 перемычек)
Parts:
- removed unit 4 of U3
- added U?: 7406, Package_DIP:DIP-14_W7.62mm_Socket, symbol 74xx_IEEE:7406
- U3: value (none) -> 7406; footprint (none) -> Package_DIP:DIP-14_W7.62mm_Socket
- U4: value (none) -> ATtiny2313V-10P; footprint (none) -> Package_DIP:DIP-20_W7.62mm
- Y1: value (none) -> 4MHz; footprint (none) -> Crystal:Crystal_HC49-4H_Vertical
Connections:
- net +5V: now also U?.14 (Vcc)
- net GNDREF: now also U?.7 (Gnd)
- net SP_1: now also U4.13 (PB1); no longer U4.19 (PB7)
- net SP_2: now also U4.15 (PB3); no longer U4.18 (PB6)
- net SP_4: now also U4.19 (PB7); no longer U4.16 (PB4)
- net SP_5: now also U4.12 (PB0); no longer U4.15 (PB3)
- net SP_7: now also U4.16 (PB4); no longer U4.13 (PB1)
- net SP_8: now also U4.18 (PB6); no longer U4.12 (PB0)
- net SP_EN: now also U?.2; no longer U3.12
- net Spin_Dir: no longer U3.11
- net Spin_En: now also U?.1; no longer U3.13
- net Spin_PWM: now also U3.11
- net at U4.6 (PD2), U4.7 (PD3): now also U3.10
- no-connect marks 7 -> 9
Other:
- moved on the sheet: U3E, U3F

Commit message: [*] Разведена плата в один слой (3 перемычки на шине 5В; 2 соединения земли через плату STM
Parts:
- gave numbers to parts that had none: 1
Connections:
- net SP_EN: now also U3.12; no longer U3.2
- net Spin_En: now also U3.13; no longer U3.1
- net Spin_PWM: now also U3.1; no longer U3.11
- net at U4.6 (PD2), U4.7 (PD3): now also U3.2; no longer U3.10
Other:
- moved on the sheet: U3A, U3E, U3F
Changed lines of the file:
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@@
     (pin "2")
   )
-  (symbol (lib_id "74xx_IEEE:7406") (at 190.5 110.49 0) (mirror y) (unit 6)
-    (in_bom yes) (on_board yes)
-    (property "Reference" "U3" (id 0) (at 194.31 102.87 0))
-    (property "Value" "7406" (id 1) (at 190.5 105.41 0))
-    (property "Footprint" "Package_DIP:DIP-14_W7.62mm_Socket" (id 2) (at 190.5 110.49 0)
-      (effects (font (size 1.27 1.27)) hide)
-    )
-    (property "Datasheet" "" (id 3) (at 190.5 110.49 0)
+  (symbol (lib_id "74xx_IEEE:7406") (at 190.5 135.89 0) (mirror y) (unit 6)
+    (in_bom yes) (on_board yes)
+    (property "Reference" "U3" (id 0) (at 194.31 128.27 0))
+    (property "Value" "7406" (id 1) (at 190.5 130.81 0))
+    (property "Footprint" "Package_DIP:DIP-14_W7.62mm_Socket" (id 2) (at 190.5 135.89 0)
+      (effects (font (size 1.27 1.27)) hide)
+    )
+    (property "Datasheet" "" (id 3) (at 190.5 135.89 0)
       (effects (font (size 1.27 1.27)) hide)
     )
@@
     (pin "1")
   )
-  (symbol (lib_id "74xx_IEEE:7406") (at 190.5 135.89 0) (mirror y) (unit 1)
-    (in_bom yes) (on_board yes)
-    (property "Reference" "U?" (id 0) (at 195.58 128.27 0))
-    (property "Value" "7406" (id 1) (at 190.5 132.08 0))
-    (property "Footprint" "Package_DIP:DIP-14_W7.62mm_Socket" (id 2) (at 190.5 135.89 0)
-      (effects (font (size 1.27 1.27)) hide)
-    )
-    (property "Datasheet" "" (id 3) (at 190.5 135.89 0)
+  (symbol (lib_id "74xx_IEEE:7406") (at 190.5 85.09 0) (mirror y) (unit 1)
+    (in_bom yes) (on_board yes)
+    (property "Reference" "U3" (id 0) (at 195.58 77.47 0))
+    (property "Value" "7406" (id 1) (at 190.5 81.28 0))
+    (property "Footprint" "Package_DIP:DIP-14_W7.62mm_Socket" (id 2) (at 190.5 85.09 0)
+      (effects (font (size 1.27 1.27)) hide)
+    )
+    (property "Datasheet" "" (id 3) (at 190.5 85.09 0)
       (effects (font (size 1.27 1.27)) hide)
     )
@@
     (pin "1")
   )
-  (symbol (lib_id "74xx_IEEE:7406") (at 190.5 85.09 0) (mirror y) (unit 5)
-    (in_bom yes) (on_board yes)
-    (property "Reference" "U3" (id 0) (at 194.31 77.47 0))
-    (property "Value" "7406" (id 1) (at 190.5 80.01 0))
-    (property "Footprint" "Package_DIP:DIP-14_W7.62mm_Socket" (id 2) (at 190.5 85.09 0)
-      (effects (font (size 1.27 1.27)) hide)
-    )
-    (property "Datasheet" "" (id 3) (at 190.5 85.09 0)
-      (effects (font (size 1.27 1.27)) hide)
-    )
+  (symbol (lib_id "74xx_IEEE:7406") (at 190.5 110.49 0) (mirror y) (unit 5)
+    (in_bom yes) (on_board yes)
+    (property "Reference" "U3" (id 0) (at 194.31 102.87 0))
+    (property "Value" "7406" (id 1) (at 190.5 105.41 0))
+    (property "Footprint" "Package_DIP:DIP-14_W7.62mm_Socket" (id 2) (at 190.5 110.49 0)
+      (effects (font (size 1.27 1.27)) hide)
+    )
+    (property "Datasheet" "" (id 3) (at 190.5 110.49 0)
+      (effects (font (size 1.27 1.27)) hide)
+    )
