File: CNC_New_ControlPlate/steppers.kicad_sch (KiCad schematic)
At the start: 5 parts

Commit message: Add spindel sch
Parts:
- C?: value (none) -> 100 pF; footprint (none) -> Capacitor_SMD:C_0603_1608Metric_Pad1.08x0.95mm_HandSolder
- D?: value (none) -> SN75ALS192N
- U? (x2): value (none) -> 7406
Changed lines of the file:
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@@
     (in_bom yes) (on_board yes)
     (property "Reference" "U?" (id 0) (at 149.86 50.8 0))
-    (property "Value" "" (id 1) (at 149.86 46.99 0)
+    (property "Value" "7406" (id 1) (at 149.86 46.99 0)
       (effects (font (size 1.27 1.27)) hide)
     )
@@
     (in_bom yes) (on_board yes)
     (property "Reference" "U?" (id 0) (at 149.86 34.29 0))
-    (property "Value" "" (id 1) (at 149.86 29.21 0))
+    (property "Value" "7406" (id 1) (at 149.86 29.21 0))
     (property "Footprint" "" (id 2) (at 149.86 39.37 0)
       (effects (font (size 1.27 1.27)) hide)
@@
     (in_bom yes) (on_board yes) (fields_autoplaced)
     (property "Reference" "D?" (id 0) (at 58.42 41.91 0))
-    (property "Value" "" (id 1) (at 58.42 44.45 0))
+    (property "Value" "SN75ALS192N" (id 1) (at 58.42 44.45 0))
     (property "Footprint" "Package_DIP:DIP-16_W7.62mm_Socket" (id 2) (at 58.42 44.45 0)
       (effects (font (size 1.27 1.27)) hide)
@@
     (in_bom yes) (on_board yes) (fields_autoplaced)
     (property "Reference" "C?" (id 0) (at 85.09 29.21 90))
-    (property "Value" "" (id 1) (at 85.09 31.75 90))
-    (property "Footprint" "" (id 2) (at 88.9 35.8648 0)
+    (property "Value" "100 pF" (id 1) (at 85.09 31.75 90))
+    (property "Footprint" "Capacitor_SMD:C_0603_1608Metric_Pad1.08x0.95mm_HandSolder" (id 2) (at 88.9 35.8648 0)
       (effects (font (size 1.27 1.27)) hide)
     )

Commit message: Add attiny2313
Parts:
- U?: value (none) -> 7406
Changed lines of the file:
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@@
     (in_bom yes) (on_board yes)
     (property "Reference" "U?" (id 0) (at 149.86 67.31 0))
-    (property "Value" "" (id 1) (at 149.86 63.5 0)
+    (property "Value" "7406" (id 1) (at 149.86 63.5 0)
       (effects (font (size 1.27 1.27)) hide)
     )

Commit message: [*] номиналы блокировочных конденсаторов [+] мкроконтроллер управления оборотами шпинделя [+] кнопка паузы
Parts:
- added C?: 100 nF, Capacitor_SMD:C_0603_1608Metric_Pad1.08x0.95mm_HandSolder, symbol Device:C
- C?: value 100 pF -> 100 nF
Connections:
- net +5V: now also C?.2
- net GNDREF: now also C?.1
Changed lines of the file:
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@@
 (kicad_sch (version 20211123) (generator eeschema)
   (paper "A5")
+  (junction (at 114.3 64.77) (diameter 0) (color 0 0 0 0)
+  )
   (junction (at 114.3 31.75) (diameter 0) (color 0 0 0 0)
   )
@@
     (stroke (width 0) (type default) (color 0 0 0 0))
   )
+  (wire (pts (xy 111.76 64.77) (xy 114.3 64.77))
+    (stroke (width 0) (type default) (color 0 0 0 0))
+  )
   (wire (pts (xy 72.39 66.04) (xy 80.01 66.04))
     (stroke (width 0) (type default) (color 0 0 0 0))
@@
     (stroke (width 0) (type default) (color 0 0 0 0))
   )
+  (wire (pts (xy 101.6 67.31) (xy 101.6 64.77))
+    (stroke (width 0) (type default) (color 0 0 0 0))
+  )
   (wire (pts (xy 90.17 36.83) (xy 90.17 50.8))
     (stroke (width 0) (type default) (color 0 0 0 0))
@@
   )
   (wire (pts (xy 72.39 68.58) (xy 80.01 68.58))
+    (stroke (width 0) (type default) (color 0 0 0 0))
+  )
+  (wire (pts (xy 101.6 64.77) (xy 104.14 64.77))
     (stroke (width 0) (type default) (color 0 0 0 0))
   )
@@
     (in_bom yes) (on_board yes) (fields_autoplaced)
     (property "Reference" "C?" (id 0) (at 85.09 29.21 90))
-    (property "Value" "100 pF" (id 1) (at 85.09 31.75 90))
+    (property "Value" "100 nF" (id 1) (at 85.09 31.75 90))
     (property "Footprint" "Capacitor_SMD:C_0603_1608Metric_Pad1.08x0.95mm_HandSolder" (id 2) (at 88.9 35.8648 0)
       (effects (font (size 1.27 1.27)) hide)
     )
     (property "Datasheet" "~" (id 3) (at 85.09 36.83 0)
+      (effects (font (size 1.27 1.27)) hide)
+    )
+    (pin "1")
+    (pin "2")
+  )
+  (symbol (lib_id "Device:C") (at 107.95 64.77 90) (unit 1)
+    (in_bom yes) (on_board yes) (fields_autoplaced)
+    (property "Reference" "C?" (id 0) (at 107.95 57.15 90))
+    (property "Value" "100 nF" (id 1) (at 107.95 59.69 90))
+    (property "Footprint" "Capacitor_SMD:C_0603_1608Metric_Pad1.08x0.95mm_HandSolder" (id 2) (at 111.76 63.8048 0)
+      (effects (font (size 1.27 1.27)) hide)
+    )
+    (property "Datasheet" "~" (id 3) (at 107.95 64.77 0)
       (effects (font (size 1.27 1.27)) hide)
     )
@@
       (effects (font (size 1.27 1.27)) hide)
     )
+    (pin "1")
+  )
+  (symbol (lib_id "power:GNDREF") (at 101.6 67.31 0) (unit 1)
+    (in_bom yes) (on_board yes) (fields_autoplaced)
+    (property "Reference" "#PWR?" (id 0) (at 101.6 73.66 0)
+      (effects (font (size 1.27 1.27)) hide)
+    )
+    (property "Value" "GNDREF" (id 1) (at 101.6 72.39 0))
+    (property "Footprint" "" (id 2) (at 101.6 67.31 0)
+      (effects (font (size 1.27 1.27)) hide)
+    )
+    (property "Datasheet" "" (id 3) (at 101.6 67.31 0)
+      (effects (font (size 1.27 1.27)) hide)
+    )
